File: zukunftroller.kicad_pcb (KiCad board)
At the start: 2 copper layers, 98 parts, among them SW1 SW_PUSH, SW10 SW_PUSH, SW11 SW_PUSH, SW12 SW_PUSH, SW13 SW_PUSH, SW14 SW_PUSH, SW15 SW_PUSH, SW16 SW_PUSH, SW17 SW_PUSH, SW18 SW_PUSH, SW19 SW_PUSH, SW2 SW_PUSH, SW20 SW_PUSH, SW21 SW_PUSH, SW22 SW_PUSH, SW23 SW_PUSH, SW24 SW_PUSH, SW25 SW_PUSH, SW26 SW_PUSH, SW27 SW_PUSH, SW28 SW_PUSH, SW29 SW_PUSH, SW3 SW_PUSH, SW30 SW_PUSH, SW31 SW_PUSH, SW32 SW_PUSH, SW33 SW_PUSH, SW34 SW_PUSH, SW35 SW_PUSH, SW36 SW_PUSH, SW37 SW_PUSH, SW38 SW_PUSH, SW39 SW_PUSH, SW4 SW_PUSH, SW40 SW_PUSH, SW41 SW_PUSH, SW42 SW_PUSH, SW43 SW_PUSH, SW44 SW_PUSH, SW45 SW_PUSH, SW46 SW_PUSH, SW47 SW_PUSH, SW48 SW_PUSH, SW5 SW_PUSH, SW6 SW_PUSH, SW7 SW_PUSH, SW8 SW_PUSH, SW9 SW_PUSH, U1 CD74HCT4067, U2 CD74HCT4067

Commit message: assigned footprints, in process of scattering elements in pcb
Parts:
- removed SW34, SW35: SW_PUSH, Buttons_Switches_ThroughHole:SW_PUSH_6mm
- added D49: D, Diodes_ThroughHole:D_A-405_P7.62mm_Horizontal, F.Cu at (15.2, -22.9)
- added D50: D, Diodes_ThroughHole:D_A-405_P7.62mm_Horizontal, F.Cu at (15.2, -17.8)
- added D51: D, Diodes_ThroughHole:D_A-405_P7.62mm_Horizontal, F.Cu at (15.2, -12.7)
- added D52: D, Diodes_ThroughHole:D_A-405_P7.62mm_Horizontal, F.Cu at (15.2, -27.9)
- added D53: D, Diodes_ThroughHole:D_A-405_P7.62mm_Horizontal, F.Cu at (15.2, -33.0)
- added D54: D, Diodes_ThroughHole:D_A-405_P7.62mm_Horizontal, F.Cu at (15.2, -38.1)
- added D55: D, Diodes_ThroughHole:D_A-405_P7.62mm_Horizontal, F.Cu at (15.2, -8.89)
- added D56: LED, LEDs:LED_D5.0mm, F.Cu at (35.6, 116.8)
- added D57: LED, LEDs:LED_D5.0mm, F.Cu at (-12.7, 50.8)
- added D58: LED, LEDs:LED_D5.0mm, F.Cu at (-12.7, 58.4)
- added D59: LED, LEDs:LED_D5.0mm, F.Cu at (-12.7, 67.3)
- added D60: LED, LEDs:LED_D5.0mm, F.Cu at (-1.27, -21.6)
- added D61: LED, LEDs:LED_D5.0mm, F.Cu at (-47.0, 8.89)
- added D62: LED, LEDs:LED_D5.0mm, F.Cu at (-72.4, -16.5)
- added D63: LED, LEDs:LED_D5.0mm, F.Cu at (-53.3, -6.35)
- added D64: LED, LEDs:LED_D5.0mm, F.Cu at (-74.9, 6.35)
- added D65: LED, LEDs:LED_D5.0mm, F.Cu at (-57.1, -20.3)
- added D66: LED, LEDs:LED_D5.0mm, F.Cu at (-50.8, -30.5)
- added D67: LED, LEDs:LED_D5.0mm, F.Cu at (-63.5, 0.00)
- added D68: LED, LEDs:LED_D5.0mm, F.Cu at (-68.6, -26.7)
- added D69: LED, LEDs:LED_D5.0mm, F.Cu at (-58.4, 14.0)
- added D70: LED, LEDs:LED_D5.0mm, F.Cu at (-62.2, -10.2)
- added D71: LED, LEDs:LED_D5.0mm, F.Cu at (-71.1, -6.35)
- added JP1: Jumper_NO_Small, SparkFun-Passives:PAD-JUMPER-2-NO_YES_SILK, F.Cu at (-2.54, 27.9)
- added JP10: Jumper_NO_Small, SparkFun-Passives:PAD-JUMPER-2-NO_YES_SILK, F.Cu at (8.89, 0.00)
- added JP11: Jumper_NO_Small, SparkFun-Passives:PAD-JUMPER-2-NO_YES_SILK, F.Cu at (31.8, 2.54)
- added JP12: Jumper_NO_Small, SparkFun-Passives:PAD-JUMPER-2-NO_YES_SILK, F.Cu at (29.2, 8.89)
- added JP13: Jumper_NO_Small, SparkFun-Passives:PAD-JUMPER-2-NO_YES_SILK, F.Cu at (-47.0, 38.1)
- added JP14: Jumper_NO_Small, SparkFun-Passives:PAD-JUMPER-2-NO_YES_SILK, F.Cu at (-44.5, 40.6)
- added JP15: Jumper_NO_Small, SparkFun-Passives:PAD-JUMPER-2-NO_YES_SILK, F.Cu at (-39.4, 45.7)
- added JP16: Jumper_NO_Small, SparkFun-Passives:PAD-JUMPER-2-NO_YES_SILK, F.Cu at (-25.4, 39.4)
- added JP17: Jumper_NO_Small, SparkFun-Passives:PAD-JUMPER-2-NO_YES_SILK, F.Cu at (-31.8, 36.8)
- added JP18: Jumper_NO_Small, SparkFun-Passives:PAD-JUMPER-2-NO_YES_SILK, F.Cu at (-19.1, 36.8)
- added JP19: Jumper_NO_Small, SparkFun-Passives:PAD-JUMPER-2-NO_YES_SILK, F.Cu at (-11.4, 35.6)
- added JP2: Jumper_NO_Small, SparkFun-Passives:PAD-JUMPER-2-NO_YES_SILK, F.Cu at (-7.62, 27.9)
- added JP3: Jumper_NO_Small, SparkFun-Passives:PAD-JUMPER-2-NO_YES_SILK, F.Cu at (2.54, 26.7)
- added JP4: Jumper_NO_Small, SparkFun-Passives:PAD-JUMPER-2-NO_YES_SILK, F.Cu at (7.62, 27.9)
- added JP5: Jumper_NO_Small, SparkFun-Passives:PAD-JUMPER-2-NO_YES_SILK, F.Cu at (2.54, 34.3)
- added JP6: Jumper_NO_Small, SparkFun-Passives:PAD-JUMPER-2-NO_YES_SILK, F.Cu at (7.62, 34.3)
- added JP7: Jumper_NO_Small, SparkFun-Passives:PAD-JUMPER-2-NO_YES_SILK, F.Cu at (-7.62, 34.3)
- added JP8: Jumper_NO_Small, SparkFun-Passives:PAD-JUMPER-2-NO_YES_SILK, F.Cu at (-1.27, 33.0)
- added JP9: Jumper_NO_Small, SparkFun-Passives:PAD-JUMPER-2-NO_YES_SILK, F.Cu at (34.3, 0.00)
- added MIDI_IN1: DIN_5, SparkFun-Connectors:DIN_5_FEMALE, F.Cu at (133.3, 40.6)
- added P1: DIN_5, SparkFun-Connectors:DIN_5_FEMALE, F.Cu at (172.7, 62.2)
- added P10: CONN_01X01, Wire_Pads:SolderWirePad_single_1-2mmDrill, F.Cu at (-27.9, 45.7)
- added P11: CONN_01X01, Wire_Pads:SolderWirePad_single_1-2mmDrill, F.Cu at (11.4, 21.6)
- added P12: CONN_01X01, Wire_Pads:SolderWirePad_single_1-2mmDrill, F.Cu at (22.9, 2.54)
- added P13: CONN_01X05, Wire_Pads:SolderWirePad_single_1-2mmDrill, F.Cu at (21.6, 25.4)
- added P14: CONN_01X05, Wire_Pads:SolderWirePad_single_1-2mmDrill, F.Cu at (-7.62, 12.7)
- added P15: CONN_01X08, Wire_Pads:SolderWirePad_single_1-2mmDrill, F.Cu at (-1.27, 16.5)
- added P16: CONN_02X03, Wire_Pads:SolderWirePad_single_1-2mmDrill, F.Cu at (25.4, 38.1)
- added P2: CONN_01_ROTARYSWITCH, SparkFun-Connectors:1X13, F.Cu at (52.1, -14.0)
- added P3: CONN_01X01, Wire_Pads:SolderWirePad_single_1-2mmDrill, F.Cu at (55.9, 2.54)
- added P4: CONN_01X01, Wire_Pads:SolderWirePad_single_1-2mmDrill, F.Cu at (47.0, 2.54)
- added P5: CONN_01X01, Wire_Pads:SolderWirePad_single_1-2mmDrill, F.Cu at (11.4, 8.89)
- added P7: CONN_01X01, Wire_Pads:SolderWirePad_single_1-2mmDrill, F.Cu at (17.8, 15.2)
- added P8: CONN_01X01, Wire_Pads:SolderWirePad_single_1-2mmDrill, F.Cu at (36.8, 17.8)
- added P9: CONN_01X01, Wire_Pads:SolderWirePad_single_1-2mmDrill, F.Cu at (-43.2, 36.8)
- added R1: R, Resistors_ThroughHole:R_Axial_DIN0309_L9.0mm_D3.2mm_P12.70mm_Horizontal, F.Cu at (-31.8, 25.4)
- added R10: R, Resistors_ThroughHole:R_Axial_DIN0309_L9.0mm_D3.2mm_P12.70mm_Horizontal, F.Cu at (-31.8, -22.9)
- added R2: R, Resistors_ThroughHole:R_Axial_DIN0309_L9.0mm_D3.2mm_P12.70mm_Horizontal, F.Cu at (-31.8, 19.1)
- added R3: R, Resistors_ThroughHole:R_Axial_DIN0309_L9.0mm_D3.2mm_P12.70mm_Horizontal, F.Cu at (-31.8, 12.7)
- added R4: R, Resistors_ThroughHole:R_Axial_DIN0309_L9.0mm_D3.2mm_P12.70mm_Horizontal, F.Cu at (-31.8, 7.62)
- added R5: R, Resistors_ThroughHole:R_Axial_DIN0309_L9.0mm_D3.2mm_P12.70mm_Horizontal, F.Cu at (-31.8, 2.54)
- added R6: R, Resistors_ThroughHole:R_Axial_DIN0309_L9.0mm_D3.2mm_P12.70mm_Horizontal, F.Cu at (-31.8, -2.54)
- added R7: R, Resistors_ThroughHole:R_Axial_DIN0309_L9.0mm_D3.2mm_P12.70mm_Horizontal, F.Cu at (-31.8, -7.62)
- added R8: R, Resistors_ThroughHole:R_Axial_DIN0309_L9.0mm_D3.2mm_P12.70mm_Horizontal, F.Cu at (-31.8, -12.7)
- added R9: R, Resistors_ThroughHole:R_Axial_DIN0309_L9.0mm_D3.2mm_P12.70mm_Horizontal, F.Cu at (-31.8, -17.8)
- added SHIELD1: ARDUINO_SHIELD, Arduino_Shields:ARDUINO SHIELD, F.Cu at (33.0, 82.5)
- added U3: 6N138, SparkFun-DigitalIC:DIL08, F.Cu at (200.7, 36.8)
- added U4: 74HC595, SparkFun-DigitalIC:DIL16, F.Cu at (74.9, 132.1)
- added U5: 74HC595, SparkFun-DigitalIC:DIL16, F.Cu at (94.0, 104.1)
- D1, D10, D11, D12, D13, D14, D15, D16, D17, D18, D19, D2, D20, D21, D22, D23, D24, D25, D26, D27, D28, D29, D3, D30, D31, D32, D33, D34, D35, D36, D37, D38, D39, D4, D40, D41, D42, D43, D44, D45, D46, D47, D48, D5, D6, D7, D8, D9: footprint Buttons_Switches_ThroughHole:SW_PUSH_6mm -> Diodes_ThroughHole:D_A-405_P7.62mm_Horizontal
- SW19, SW5: value SW_PUSH -> ROTARY_ENCODER; footprint Buttons_Switches_ThroughHole:SW_PUSH_6mm -> SparkFun-Electromechanical:ENCODER_LED_2
- SW20: value SW_PUSH -> SWITCH_INV; footprint Buttons_Switches_ThroughHole:SW_PUSH_6mm -> SparkFun-Electromechanical:SWITCH-SPDT
Connections:
- D19 pad 1: /MUXB_CONN_1 -> /MUXA_CONN_1
- D20 pad 1: /MUXB_CONN_1 -> /MUXA_CONN_2
- D34 pad 1: /MUXB_CONN_0 -> /MUXA_CONN_3
- D35 pad 1: /MUXB_CONN_0 -> /MUXA_CONN_4
- D4 pad 1: /MUXB_CONN_2 -> Net-(D4-Pad1)
- D5 pad 1: /MUXB_CONN_2 -> /MUXA_CONN_0
- SW20 pad 1: /MUXA_CONN_E -> /MUXB_CONN_7
- SW20 pad 2: Net-(D20-Pad2) -> GND
- SW4 pad 1: /MUXA_CONN_F -> /RESET
- SW4 pad 2: Net-(D4-Pad2) -> GND
- U1 pad 12: Net-(U1-Pad12) -> (no net)
- U1 pad 15: /MUXA_INHIBIT -> GND
- U1 pad 24: Net-(U1-Pad24) -> (no net)
- U2 pad 12: Net-(U2-Pad12) -> (no net)
- U2 pad 15: /MUXB_INHIBIT -> GND
- U2 pad 16: /MUXB_CONN_F -> (no net)
- U2 pad 17: /MUXB_CONN_E -> (no net)
- U2 pad 19: /MUXB_CONN_C -> (no net)
- U2 pad 20: /MUXB_CONN_B -> (no net)
- U2 pad 21: /MUXB_CONN_A -> (no net)
- U2 pad 22: /MUXB_CONN_9 -> (no net)
- U2 pad 24: Net-(U2-Pad24) -> (no net)

Commit message: sorting buttons, changed footprint of 4067
Parts:
- U1, U2: footprint SparkFun-PowerIC:SSOP24 -> SparkFun-DigitalIC:DIL24-6
- moved SW33 419.3 mm to (104.1, 522.0)
- moved SW48 378.0 mm to (43.0, 467.9)
- moved D19 366.3 mm to (168.9, 509.3)
- moved SW18 354.1 mm to (127.0, 458.5)
- moved D15 292.8 mm to (87.6, 375.9)
- moved SW45 289.2 mm to (62.1, 381.0)
- moved D45 281.9 mm to (62.2, 373.4)
- moved SW15 281.7 mm to (88.9, 380.3)
- moved SW30 274.7 mm to (111.6, 377.2)
- moved SW39 263.6 mm to (373.4, 242.6)
- moved SW40 258.4 mm to (69.7, 351.1)
- moved SW16 254.6 mm to (382.3, 205.7)
- moved SW10 253.5 mm to (87.6, 351.1)
- moved D40 253.4 mm to (68.6, 345.4)
- moved SW25 249.5 mm to (111.8, 351.8)
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
Commit message: more sorting
Parts:
- moved SW13 377.3 mm to (86.2, 459.1)
- moved D20 361.8 mm to (88.9, 421.6)
- moved SW17 360.0 mm to (88.9, 408.9)
- moved SW28 317.5 mm to (107.8, 453.4)
- moved SW43 305.5 mm to (68.4, 464.8)
- moved SW47 260.1 mm to (67.2, 407.0)
- moved D47 246.2 mm to (67.3, 419.1)
- moved SW32 237.2 mm to (118.0, 410.2)
- moved D43 232.7 mm to (67.3, 449.6)
- moved D32 225.5 mm to (115.6, 422.9)
- moved D13 224.8 mm to (85.1, 452.1)
- moved D28 184.8 mm to (105.4, 442.0)
- moved SW18 30.7 mm to (106.5, 481.3)
Changed lines of the file:
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@@
   )
   (module Buttons_Switches_ThroughHole:SW_PUSH_6mm (layer F.Cu)
-    (at 328.93 170.18)
+    (at 86.21 459.05)
     (descr https://www.omron.com/ecb/products/pdf/en-b3f.pdf)
     (tags "tact sw push 6mm")
@@
   )
   (module Buttons_Switches_ThroughHole:SW_PUSH_6mm (layer F.Cu)
-    (at 367.03 180.34)
+    (at 88.9 408.94)
     (descr https://www.omron.com/ecb/products/pdf/en-b3f.pdf)
     (tags "tact sw push 6mm")
@@
   )
   (module Buttons_Switches_ThroughHole:SW_PUSH_6mm (layer F.Cu)
-    (at 127 458.47)
+    (at 106.53 481.33)
     (descr https://www.omron.com/ecb/products/pdf/en-b3f.pdf)
     (tags "tact sw push 6mm")
@@
   )
   (module Buttons_Switches_ThroughHole:SW_PUSH_6mm (layer F.Cu)
-    (at 321.31 218.44)
+    (at 107.8 453.39)
     (descr https://www.omron.com/ecb/products/pdf/en-b3f.pdf)
     (tags "tact sw push 6mm")
@@
   )
   (module Buttons_Switches_ThroughHole:SW_PUSH_6mm (layer F.Cu)
-    (at 270.51 228.6)
+    (at 117.96 410.21)
     (descr https://www.omron.com/ecb/products/pdf/en-b3f.pdf)
     (tags "tact sw push 6mm")
@@
   )
   (module Buttons_Switches_ThroughHole:SW_PUSH_6mm (layer F.Cu)
-    (at 279.4 243.84)
+    (at 68.43 464.82)
     (descr https://www.omron.com/ecb/products/pdf/en-b3f.pdf)
     (tags "tact sw push 6mm")
@@
   )
   (module Buttons_Switches_ThroughHole:SW_PUSH_6mm (layer F.Cu)
-    (at 254 226.06)
+    (at 67.16 406.98)
     (descr https://www.omron.com/ecb/products/pdf/en-b3f.pdf)
     (tags "tact sw push 6mm")
@@
   )
   (module Diodes_ThroughHole:D_A-405_P7.62mm_Horizontal (layer F.Cu)
-    (at 85.09 227.33)
+    (at 85.09 452.12)
     (descr "D, A-405 series, Axial, Horizontal, pin pitch=7.62mm, , length*diameter=5.2*2.7mm^2, , http://www.diodes.com/_files/packages/A-405.pdf")
     (tags "D A-405 series Axial Horizontal pin pitch 7.62mm  length 5.2mm diameter 2.7mm")
@@
   )
   (module Diodes_ThroughHole:D_A-405_P7.62mm_Horizontal (layer F.Cu)
-    (at 392.43 224.79)
+    (at 88.9 421.64)
     (descr "D, A-405 series, Axial, Horizontal, pin pitch=7.62mm, , length*diameter=5.2*2.7mm^2, , http://www.diodes.com/_files/packages/A-405.pdf")
     (tags "D A-405 series Axial Horizontal pin pitch 7.62mm  length 5.2mm diameter 2.7mm")
@@
   )
   (module Diodes_ThroughHole:D_A-405_P7.62mm_Horizontal (layer F.Cu)
-    (at 120.65 257.81)
+    (at 105.41 441.96)
     (descr "D, A-405 series, Axial, Horizontal, pin pitch=7.62mm, , length*diameter=5.2*2.7mm^2, , http://www.diodes.com/_files/packages/A-405.pdf")
     (tags "D A-405 series Axial Horizontal pin pitch 7.62mm  length 5.2mm diameter 2.7mm")
@@
   )
   (module Diodes_ThroughHole:D_A-405_P7.62mm_Horizontal (layer F.Cu)
-    (at 120.65 197.485)
+    (at 115.57 422.91)
     (descr "D, A-405 series, Axial, Horizontal, pin pitch=7.62mm, , length*diameter=5.2*2.7mm^2, , http://www.diodes.com/_files/packages/A-405.pdf")
     (tags "D A-405 series Axial Horizontal pin pitch 7.62mm  length 5.2mm diameter 2.7mm")
@@
   )
   (module Diodes_ThroughHole:D_A-405_P7.62mm_Horizontal (layer F.Cu)
-    (at 55.88 217.16)
+    (at 67.31 449.58)
     (descr "D, A-405 series, Axial, Horizontal, pin pitch=7.62mm, , length*diameter=5.2*2.7mm^2, , http://www.diodes.com/_files/packages/A-405.pdf")
     (tags "D A-405 series Axial Horizontal pin pitch 7.62mm  length 5.2mm diameter 2.7mm")
@@
   )
   (module Diodes_ThroughHole:D_A-405_P7.62mm_Horizontal (layer F.Cu)
-    (at 55.88 173.12)
+    (at 67.31 419.1)
     (descr "D, A-405 series, Axial, Horizontal, pin pitch=7.62mm, , length*diameter=5.2*2.7mm^2, , http://www.diodes.com/_files/packages/A-405.pdf")
     (tags "D A-405 series Axial Horizontal pin pitch 7.62mm  length 5.2mm diameter 2.7mm")
